Commit message: Placing some reasonable-enough joint bounds

File: excavatorURDF/robot_fixed_alternate.urdf (robot description, URDF)
Before this commit: robot onshape, 19 links, 18 joints
Joints:
- joint full_arm_rotation: limit effort=1 velocity=20 -> lower=-0.1 upper=0.8 effort=1 velocity=20
- joint idler1_wheel: type continuous -> fixed
- joint idler2_wheel: type continuous -> fixed
- joint left_idle_passive_wheel: type continuous -> fixed
- joint left_sprocket_wheel: type continuous -> fixed
- joint lower_arm: limit effort=1 velocity=20 -> lower=-0.4 upper=1.0 effort=1 velocity=20
- joint right_idle_passive_wheel: type continuous -> fixed
- joint right_sprocket_wheel: type continuous -> fixed
- joint roll_wheel_1: type continuous -> fixed
- joint roll_wheel_2: type continuous -> fixed
- joint roll_wheel_3: type continuous -> fixed
- joint roll_wheel_4: type continuous -> fixed
- joint roll_wheel_5: type continuous -> fixed
- joint roll_wheel_6: type continuous -> fixed
- joint upperToLow: limit effort=1 velocity=20 -> lower=-0.9 upper=0.3 effort=1 velocity=20

Commit message: Some largely minor changes

File: excavatorURDF/robot_fixed_alternate.urdf (robot description, URDF)
Before this commit: robot onshape, 19 links, 18 joints
Joints:
- joint lower_arm: limit lower=-0.4 upper=1.0 effort=1 velocity=20 -> lower=-0.4 upper=1.0 effort=12 velocity=20
- joint tankSpin_wheel: limit effort=1 velocity=20 -> effort=1 velocity=5
- joint upperToLow: limit lower=-0.9 upper=0.3 effort=1 velocity=20 -> lower=-0.9 upper=0.3 effort=5 velocity=20

Commit message: Scheme modifications for floating action

File: excavatorURDF/robot_fixed_alternate.urdf (robot description, URDF)
Before this commit: robot onshape, 19 links, 18 joints
Joints:
- joint full_arm_rotation: limit lower=-0.1 upper=0.8 effort=1 velocity=20 -> lower=-0.1 upper=0.8 effort=10000 velocity=1
- joint lower_arm: limit lower=-0.4 upper=1.0 effort=12 velocity=20 -> lower=-0.45 upper=1.0 effort=40000 velocity=.8
- joint scoop1: limit lower=-1.2217304763960306069 upper=0.87266462599716476678 effort=1 velocity=20 -> lower=-1.2217304763960306069 upper=0.87266462599716476678 effort=10000 velocity=3
- joint tankSpin_wheel: limit effort=1 velocity=5 -> effort=20000 velocity=1
- joint upperToLow: limit lower=-0.9 upper=0.3 effort=5 velocity=20 -> lower=-0.9 upper=0.3 effort=20000 velocity=1.5
