Commit message: Excavator simulation prototyping - still somewhat slow and some moderate leaking

File: excavatorURDF/excavator_boxy_locked.urdf (robot description, URDF)
Before this commit: robot onshape, 19 links, 18 joints
Links:
- link part04: geometry collision box size=0.170 0.600 0.650; collision box size=0.170 0.700 0.650
Joints:
- joint full_arm_rotation: limit lower=-0.1 upper=0.8 effort=10000 velocity=1 -> (none); origin xyz=-0.040707723917193440466 -0.80673603465099630316 0.38039999999999996039 rpy=3.141592653589793116 1.3405772267554363358e-16 0.49184482936957452104 -> xyz=-0.040707723917193440466 -0.80673603465099630316 0.38039999999999996039 rpy=3.141592653589793116 1.3405772267554363358e-16 0; type revolute -> fixed
- joint lower_arm: limit lower=-0.45 upper=1.0 effort=40000 velocity=.8 -> lower=-0.45 upper=1.0 effort=40000 velocity=.45
- joint scoop1: limit lower=-1.2217304763960306069 upper=0.87266462599716476678 effort=10000 velocity=3 -> lower=-1.2217304763960306069 upper=0.87266462599716476678 effort=10000 velocity=0.7
- joint tankSpin_wheel: limit effort=20000 velocity=1 -> effort=20000 velocity=1.1
- joint upperToLow: limit lower=-0.9 upper=0.3 effort=20000 velocity=1.5 -> lower=-0.9 upper=0.3 effort=20000 velocity=.45

File: excavatorURDF/excavator_prototype_mulitway_box.urdf (robot description, URDF)
Before this commit: robot onshape, 19 links, 18 joints
Links:
- link part04: geometry collision box size=0.090 0.240 0.680; collision box size=0.185 0.615 0.680
