Commit message: Cut-back simulator for pre-generated replays only

File: excavatorURDF/excavator_lowpoly_locked.urdf (robot description, URDF)
Before this commit: robot onshape, 19 links, 18 joints
Links:
- removed link part04
- added link bucketry, mass 132.60396921004004867; collision mesh filename=bucket_low_poly_no_interior.stl; collision mesh filename=bucket_mount.stl
Joints:
- joint scoop1: child part04 -> bucketry

File: excavatorURDF/excavator_lowpoly_locked_splitbucket.urdf (robot description, URDF)
Before this commit: robot onshape, 19 links, 18 joints
Links:
- removed link part02_cmpl
- removed link part03
- removed link part04
- added link bucketry, mass 132.60396921004004867; collision mesh filename=bucket_floor.stl; collision mesh filename=bucket_left.stl
- added link lower_boom, mass 265.34907807560870197; collision mesh filename=part03.stl; visual mesh filename=part03.stl
- added link upper_boom, mass 694.17793513858077858; collision mesh filename=part02.stl; visual mesh filename=part02.stl
Joints:
- joint full_arm_rotation: origin xyz=-0.040707723917193440466 -0.80673603465099630316 0.38039999999999996039 rpy=3.141592653589793116 1.3405772267554363358e-16 0 -> xyz=-0.040707723917193440466 -0.80673603465099630316 0.38039999999999996039 rpy=3.141592653589793116 0 0
- joint lower_arm: child part02_cmpl -> upper_boom
- joint scoop1: child part04 -> bucketry; parent part03 -> lower_boom
- joint upperToLow: child part03 -> lower_boom; parent part02_cmpl -> upper_boom
