Commit message: These buckets are the best we'll be able to get

File: excavatorURDF/excavator_lowpoly_locked_splitbucket.urdf (robot description, URDF)
Before this commit: robot onshape, 19 links, 18 joints
Links:
- link part04: geometry collision mesh filename=bucket_floor.stl; collision mesh filename=bucket_left.stl

Commit message: Some final merging / cleaning

File: excavatorURDF/excavator_lowpoly_locked_splitbucket.urdf (robot description, URDF)
Before this commit: robot onshape, 19 links, 18 joints
Joints:
- joint full_arm_rotation: origin xyz=-0.040707723917193440466 -0.80673603465099630316 0.38039999999999996039 rpy=3.141592653589793116 0 0 -> xyz=-0.04 -0.8 0.38 rpy=3.141592653589793116 0 0
- joint lower_arm: origin xyz=0.079999999999999904521 0.074999999999999733546 -0.14999999999999980016 rpy=-1.570796326794896558 0.69362897114705091006 -1.5707963267948985564 -> xyz=0.08 0.075 -0.15 rpy=-1.57 0.7 -1.57
- joint scoop1: origin xyz=0.11999999999999966249 -1.5403327562575594989 -3.8857805861880478915e-16 rpy=3.1415926535897895633 -3.1950791765547316365e-15 -0.80531265657487949294 -> xyz=0.12 -1.54 0 rpy=3.1415926535897895633 0 -0.805
- joint upperToLow: origin xyz=-0.83999999999999985789 2.3549999999999999822 -0.13499999999999978684 rpy=-3.1415926535897877869 -7.0950929862569758372e-15 1.2267499240314121423 -> xyz=-0.84 2.355 -0.135 rpy=-3.1415926535897877869 0 1.23
